File: uv-lamp.kicad_pcb (KiCad board)
At the start: 2 copper layers, 133 parts, among them J1 Conn, J2 Barrel_Jack_Switch, J3 Jmp, Q1 STN4NF20L, Q2 STN4NF20L, Q3 STN4NF20L, Q4 STN4NF20L, Q5 FDD120AN15A0, U1 MP3394S

Commit message: ...
Routing:
- net /LED/C4: track 334.0 -> 353.5 mm
- net /LED/C1: track 330.3 -> 346.8 mm
- net Net-(D47-Pad1): track 29.0 -> 16.7 mm
- net Net-(D17-Pad1): track 29.0 -> 16.7 mm
- net Net-(D57-Pad1): track 25.9 -> 14.3 mm
- net Net-(D29-Pad1): track 25.9 -> 14.3 mm
- net Net-(D59-Pad1): track 25.9 -> 15.3 mm
- net Net-(D31-Pad1): track 25.9 -> 15.3 mm
- net Net-(D19-Pad1): track 31.5 -> 21.7 mm
- net Net-(D45-Pad1): track 29.1 -> 19.3 mm
- net Net-(D30-Pad1): track 29.0 -> 25.7 mm
- net Net-(D75-Pad1): track 26.3 -> 29.1 mm
- net Net-(D58-Pad1): track 29.0 -> 26.7 mm
- net Net-(D40-Pad1): track 25.4 -> 27.0 mm
- net /SMPS/VMOSA: track 181.7 -> 183.2 mm
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
Commit message: Update uv-lamp.kicad_pcb
Parts:
- moved C6 7.00 mm to (271.5, 44.5)
- moved C3 6.25 mm to (268.8, 44.5)
- moved C8 4.30 mm to (275.5, 44.5)
- moved J2 3.31 mm to (278.8, 27.9)
- moved D1 1.75 mm to (278.9, 35.5)
- moved F1 1.75 mm to (270.8, 34.8)
- moved R18 0.60 mm to (282.8, 50.0)
- moved D3 0.56 mm to (264.2, 99.1)
Routing:
- net +12V: track 16.6 -> 15.7 mm
