File: uv-lamp.kicad_pcb (KiCad board)
At the start: 2 copper layers, 133 parts, among them J1 Conn, J2 Barrel_Jack_Switch, J3 Jmp, Q1 STN4NF20L, Q2 STN4NF20L, Q3 STN4NF20L, Q4 STN4NF20L, Q5 FDD120AN15A0, U1 MP3394S

Commit message: ...
Parts:
- C1, C2, C3: footprint Capacitors_SMD:C_1206_HandSoldering -> mod:C_1206_HandSoldering
- C4, C7, C8, C9: footprint Capacitors_SMD:C_1812_HandSoldering -> mod:C_1812_HandSoldering
- C5, C6: footprint Capacitors_SMD:C_1210_HandSoldering -> mod:C_1210_HandSoldering
- D1: footprint Diodes_SMD:D_SMB_Handsoldering -> mod:D_SMB_Handsoldering
- D2, D88, D90: footprint Diodes_SMD:D_MiniMELF_Handsoldering -> mod:D_MiniMELF_Handsoldering
- D3: footprint Diodes_SMD:D_SMC_Handsoldering -> mod:D_SMC_Handsoldering
- F1: footprint Capacitors_THT:C_Rect_L7.0mm_W2.5mm_P5.00mm -> mod:C_Rect_L7.0mm_W2.5mm_P5.00mm
- H1, H11, H12, H2: footprint Mounting_Holes:MountingHole_4.3mm_M4_Pad -> mod:MountingHole_4.3mm_M4_Pad
- J1: footprint Pin_Headers:Pin_Header_Straight_2x03_Pitch2.54mm -> mod:Pin_Header_Straight_2x03_Pitch2.54mm
- J2: footprint Connectors:BARREL_JACK -> mod:BARREL_JACK
- J3: footprint Pin_Headers:Pin_Header_Straight_2x02_Pitch2.54mm -> mod:Pin_Header_Straight_2x02_Pitch2.54mm
- L1: footprint Inductors_SMD:L_12x12mm_h8mm -> mod:L_12x12mm_h8mm
- Q1, Q2, Q3, Q4: footprint TO_SOT_Packages_SMD:SOT-223-3_TabPin2 -> mod:SOT-223-3_TabPin2
- Q5: footprint TO_SOT_Packages_SMD:TO-252-2 -> Package_TO_SOT_SMD:TO-252-2
- R1, R10, R11, R12, R14, R16, R2, R20, R3, R4, R5, R6, R7, R8, R9: footprint Resistors_SMD:R_1206_HandSoldering -> mod:R_1206_HandSoldering
- R13: footprint Resistors_SMD:R_2512_HandSoldering -> mod:R_2512_HandSoldering
- R15, R17, R18, R19: footprint Resistors_SMD:R_2010_HandSoldering -> mod:R_2010_HandSoldering
- U1: footprint Housings_SOIC:SOIC-16_3.9x9.9mm_Pitch1.27mm -> mod:SOIC-16_3.9x9.9mm_Pitch1.27mm
