File: SMPS.sch (KiCad schematic (older format))
At the start: 31 parts, among them Q1 STN4NF20L, Q2 STN4NF20L, Q3 STN4NF20L, Q4 STN4NF20L, Q5 FDD120AN15A0, U1 MP3394S

Commit message: ...
Parts:
- C1, C2: footprint Capacitors_SMD:C_1206_HandSoldering -> mod:C_1206_HandSoldering
- C4, C7, C9: footprint Capacitors_SMD:C_1812_HandSoldering -> mod:C_1812_HandSoldering
- C5: footprint Capacitors_SMD:C_1210_HandSoldering -> mod:C_1210_HandSoldering
- D2, D90: footprint Diodes_SMD:D_MiniMELF_Handsoldering -> mod:D_MiniMELF_Handsoldering
- D3: footprint Diodes_SMD:D_SMC_Handsoldering -> mod:D_SMC_Handsoldering
- L1: footprint Inductors_SMD:L_12x12mm_h8mm -> mod:L_12x12mm_h8mm
- Q1, Q2, Q3, Q4: footprint TO_SOT_Packages_SMD:SOT-223-3_TabPin2 -> mod:SOT-223-3_TabPin2
- Q5: footprint TO_SOT_Packages_SMD:TO-252-2 -> Package_TO_SOT_SMD:TO-252-2
- R10, R11, R12, R16, R2, R20, R3, R4, R5, R7, R8, R9: footprint Resistors_SMD:R_1206_HandSoldering -> mod:R_1206_HandSoldering
- R13: footprint Resistors_SMD:R_2512_HandSoldering -> mod:R_2512_HandSoldering
- R15, R17: footprint Resistors_SMD:R_2010_HandSoldering -> mod:R_2010_HandSoldering
- U1: footprint Housings_SOIC:SOIC-16_3.9x9.9mm_Pitch1.27mm -> mod:SOIC-16_3.9x9.9mm_Pitch1.27mm
Changed lines of the file:
@@
 EESchema Schematic File Version 4
-LIBS:uv-lamp-cache
-EELAYER 26 0
+EELAYER 30 0
 EELAYER END
 $Descr A4 11693 8268
@@
 F 0 "U1" H 3400 3294 40  0000 C CNN
 F 1 "MP3394S" H 3400 3218 40  0000 C CNN
-F 2 "Housings_SOIC:SOIC-16_3.9x9.9mm_Pitch1.27mm" H 3400 2550 60  0001 C CNN
+F 2 "mod:SOIC-16_3.9x9.9mm_Pitch1.27mm" H 3400 2550 60  0001 C CNN
 F 3 "" H 3400 2550 60  0000 C CNN
 	1    3400 2550
@@
 F 0 "L1" V 4240 1550 50  0000 C CNN
 F 1 "22u" V 4149 1550 50  0000 C CNN
-F 2 "Inductors_SMD:L_12x12mm_h8mm" H 4050 1550 50  0001 C CNN
+F 2 "mod:L_12x12mm_h8mm" H 4050 1550 50  0001 C CNN
 F 3 "~" H 4050 1550 50  0001 C CNN
 	1    4050 1550
@@
 F 0 "R8" H 2970 1846 50  0000 L CNN
 F 1 "4.7" H 2970 1755 50  0000 L CNN
-F 2 "Resistors_SMD:R_1206_HandSoldering" V 2830 1800 50  0001 C CNN
+F 2 "mod:R_1206_HandSoldering" V 2830 1800 50  0001 C CNN
 F 3 "~" H 2900 1800 50  0001 C CNN
 	1    2900 1800
@@
 F 0 "Q5" H 4406 1996 50  0000 L CNN
 F 1 "FDD120AN15A0" H 4406 1905 50  0000 L CNN
-F 2 "TO_SOT_Packages_SMD:TO-252-2" H 4400 2050 50  0001 C CNN
+F 2 "Package_TO_SOT_SMD:TO-252-2" H 4400 2050 50  0001 C CNN
 F 3 "~" H 4200 1950 50  0001 C CNN
 	1    4200 1950
@@
 F 0 "R11" H 5970 2596 50  0000 L CNN
 F 1 "10k" H 5970 2505 50  0000 L CNN
-F 2 "Resistors_SMD:R_1206_HandSoldering" V 5830 2550 50  0001 C CNN
+F 2 "mod:R_1206_HandSoldering" V 5830 2550 50  0001 C CNN
 F 3 "~" H 5900 2550 50  0001 C CNN
 	1    5900 2550
@@
 F 0 "D3" H 4550 1334 50  0000 C CNN
 F 1 "SS510" H 4550 1425 50  0000 C CNN
-F 2 "Diodes_SMD:D_SMC_Handsoldering" H 4550 1550 50  0001 C CNN
+F 2 "mod:D_SMC_Handsoldering" H 4550 1550 50  0001 C CNN
 F 3 "~" H 4550 1550 50  0001 C CNN
 	1    4550 1550
@@
 F 0 "R13" H 4620 2296 50  0000 L CNN
 F 1 "50m" H 4620 2205 50  0000 L CNN
-F 2 "Resistors_SMD:R_2512_HandSoldering" V 4480 2250 50  0001 C CNN
+F 2 "mod:R_2512_HandSoldering" V 4480 2250 50  0001 C CNN
 F 3 "~" H 4550 2250 50  0001 C CNN
 	1    4550 2250
@@
 F 0 "C7" H 8115 1946 50  0000 L CNN
 F 1 "4.7u" H 8115 1855 50  0000 L CNN
-F 2 "Capacitors_SMD:C_1812_HandSoldering" H 8038 1750 50  0001 C CNN
+F 2 "mod:C_1812_HandSoldering" H 8038 1750 50  0001 C CNN
 F 3 "~" H 8000 1900 50  0001 C CNN
 	1    8000 1900
@@
 F 0 "C5" H 7885 1004 50  0000 R CNN
 F 1 "4.7u" H 7885 1095 50  0000 R CNN
-F 2 "Capacitors_SMD:C_1210_HandSoldering" H 8038 900 50  0001 C CNN
+F 2 "mod:C_1210_HandSoldering" H 8038 900 50  0001 C CNN
 F 3 "~" H 8000 1050 50  0001 C CNN
 	1    8000 1050
@@
 F 0 "C1" H 2085 1754 50  0000 R CNN
 F 1 "470n" H 2085 1845 50  0000 R CNN
-F 2 "Capacitors_SMD:C_1206_HandSoldering" H 2238 1650 50  0001 C CNN
+F 2 "mod:C_1206_HandSoldering" H 2238 1650 50  0001 C CNN
 F 3 "~" H 2200 1800 50  0001 C CNN
 	1    2200 1800
@@
 F 0 "R4" H 2130 2054 50  0000 R CNN
 F 1 "270" H 2130 2145 50  0000 R CNN
-F 2 "Resistors_SMD:R_1206_HandSoldering" V 2130 2100 50  0001 C CNN
+F 2 "mod:R_1206_HandSoldering" V 2130 2100 50  0001 C CNN
 F 3 "~" H 2200 2100 50  0001 C CNN
 	1    2200 2100
@@
 F 0 "R3" H 2270 3346 50  0000 L CNN
 F 1 "120k" H 2270 3255 50  0000 L CNN
-F 2 "Resistors_SMD:R_1206_HandSoldering" V 2130 3300 50  0001 C CNN
+F 2 "mod:R_1206_HandSoldering" V 2130 3300 50  0001 C CNN
 F 3 "~" H 2200 3300 50  0001 C CNN
 	1    2200 3300
@@
 F 0 "R2" H 1070 3996 50  0000 L CNN
 F 1 "20k" H 1070 3905 50  0000 L CNN
-F 2 "Resistors_SMD:R_1206_HandSoldering" V 930 3950 50  0001 C CNN
+F 2 "mod:R_1206_HandSoldering" V 930 3950 50  0001 C CNN
 F 3 "~" H 1000 3950 50  0001 C CNN
 	1    1000 3950
@@
 F 0 "R7" H 1420 3996 50  0000 L CNN
 F 1 "20k" H 1420 3905 50  0000 L CNN
-F 2 "Resistors_SMD:R_1206_HandSoldering" V 1280 3950 50  0001 C CNN
+F 2 "mod:R_1206_HandSoldering" V 1280 3950 50  0001 C CNN
 F 3 "~" H 1350 3950 50  0001 C CNN
 	1    1350 3950
@@
 F 0 "R5" H 2620 3346 50  0000 L CNN
 F 1 "100k" H 2620 3255 50  0000 L CNN
-F 2 "Resistors_SMD:R_1206_HandSoldering" V 2480 3300 50  0001 C CNN
+F 2 "mod:R_1206_HandSoldering" V 2480 3300 50  0001 C CNN
 F 3 "~" H 2550 3300 50  0001 C CNN
 	1    2550 3300
@@
 F 0 "R9" H 2970 3346 50  0000 L CNN
 F 1 "7.5k" H 2970 3255 50  0000 L CNN
-F 2 "Resistors_SMD:R_1206_HandSoldering" V 2830 3300 50  0001 C CNN
+F 2 "mod:R_1206_HandSoldering" V 2830 3300 50  0001 C CNN
 F 3 "~" H 2900 3300 50  0001 C CNN
 	1    2900 3300
@@
 F 0 "C9" H 8565 1946 50  0000 L CNN
 F 1 "22u" H 8565 1855 50  0000 L CNN
-F 2 "Capacitors_SMD:C_1812_HandSoldering" H 8488 1750 50  0001 C CNN
+F 2 "mod:C_1812_HandSoldering" H 8488 1750 50  0001 C CNN
 F 3 "~" H 8450 1900 50  0001 C CNN
 	1    8450 1900
@@
 F 0 "C4" H 7665 1946 50  0000 L CNN
 F 1 "470n" H 7665 1855 50  0000 L CNN
-F 2 "Capacitors_SMD:C_1812_HandSoldering" H 7588 1750 50  0001 C CNN
+F 2 "mod:C_1812_HandSoldering" H 7588 1750 50  0001 C CNN
 F 3 "~" H 7550 1900 50  0001 C CNN
 	1    7550 1900
@@
 F 0 "C2" H 7665 1096 50  0000 L CNN
 F 1 "220n" H 7665 1005 50  0000 L CNN
-F 2 "Capacitors_SMD:C_1206_HandSoldering" H 7588 900 50  0001 C CNN
+F 2 "mod:C_1206_HandSoldering" H 7588 900 50  0001 C CNN
 F 3 "~" H 7550 1050 50  0001 C CNN
 	1    7550 1050
@@
 F 0 "R12" V 5143 2300 50  0000 C CNN
 F 1 "820k" V 5234 2300 50  0000 C CNN
-F 2 "Resistors_SMD:R_1206_HandSoldering" V 5280 2300 50  0001 C CNN
+F 2 "mod:R_1206_HandSoldering" V 5280 2300 50  0001 C CNN
 F 3 "~" H 5350 2300 50  0001 C CNN
 	1    5350 2300
@@
 F 0 "Q1" H 4206 3704 50  0000 L CNN
 F 1 "STN4NF20L" H 4206 3795 50  0000 L CNN
-F 2 "TO_SOT_Packages_SMD:SOT-223-3_TabPin2" H 4200 3850 50  0001 C CNN
+F 2 "mod:SOT-223-3_TabPin2" H 4200 3850 50  0001 C CNN
 F 3 "~" H 4000 3750 50  0001 C CNN
 	1    4000 3750
@@
 F 0 "Q2" H 4806 3704 50  0000 L CNN
 F 1 "STN4NF20L" H 4806 3795 50  0000 L CNN
-F 2 "TO_SOT_Packages_SMD:SOT-223-3_TabPin2" H 4800 3850 50  0001 C CNN
+F 2 "mod:SOT-223-3_TabPin2" H 4800 3850 50  0001 C CNN
 F 3 "~" H 4600 3750 50  0001 C CNN
 	1    4600 3750
@@
 F 0 "Q3" H 6106 3704 50  0000 L CNN
 F 1 "STN4NF20L" H 6106 3795 50  0000 L CNN
-F 2 "TO_SOT_Packages_SMD:SOT-223-3_TabPin2" H 6100 3850 50  0001 C CNN
+F 2 "mod:SOT-223-3_TabPin2" H 6100 3850 50  0001 C CNN
 F 3 "~" H 5900 3750 50  0001 C CNN
 	1    5900 3750
@@
 F 0 "Q4" H 6706 3704 50  0000 L CNN
 F 1 "STN4NF20L" H 6706 3795 50  0000 L CNN
-F 2 "TO_SOT_Packages_SMD:SOT-223-3_TabPin2" H 6700 3850 50  0001 C CNN
+F 2 "mod:SOT-223-3_TabPin2" H 6700 3850 50  0001 C CNN
 F 3 "~" H 6500 3750 50  0001 C CNN
 	1    6500 3750
@@
 F 0 "D2" V 4254 4079 50  0000 L CNN
 F 1 "ZMM18" V 4345 4079 50  0000 L CNN
-F 2 "Diodes_SMD:D_MiniMELF_Handsoldering" H 4300 4000 50  0001 C CNN
+F 2 "mod:D_MiniMELF_Handsoldering" H 4300 4000 50  0001 C CNN
 F 3 "~" H 4300 4000 50  0001 C CNN
 	1    4300 4000
@@
 F 0 "R10" H 4370 3546 50  0000 L CNN
 F 1 "2.2k" H 4370 3455 50  0000 L CNN
-F 2 "Resistors_SMD:R_1206_HandSoldering" V 4230 3500 50  0001 C CNN
+F 2 "mod:R_1206_HandSoldering" V 4230 3500 50  0001 C CNN
 F 3 "~" H 4300 3500 50  0001 C CNN
 	1    4300 3500
@@
 F 0 "D90" V 6154 4079 50  0000 L CNN
 F 1 "ZMM18" V 6245 4079 50  0000 L CNN
-F 2 "Diodes_SMD:D_MiniMELF_Handsoldering" H 6200 4000 50  0001 C CNN
+F 2 "mod:D_MiniMELF_Handsoldering" H 6200 4000 50  0001 C CNN
 F 3 "~" H 6200 4000 50  0001 C CNN
 	1    6200 4000
@@
 F 0 "R16" H 6270 3546 50  0000 L CNN
 F 1 "2.2k" H 6270 3455 50  0000 L CNN
-F 2 "Resistors_SMD:R_1206_HandSoldering" V 6130 3500 50  0001 C CNN
+F 2 "mod:R_1206_HandSoldering" V 6130 3500 50  0001 C CNN
 F 3 "~" H 6200 3500 50  0001 C CNN
 	1    6200 3500
@@
 F 0 "R15" H 5870 3146 50  0000 L CNN
 F 1 "0" H 5870 3055 50  0000 L CNN
-F 2 "Resistors_SMD:R_2010_HandSoldering" V 5730 3100 50  0001 C CNN
+F 2 "mod:R_2010_HandSoldering" V 5730 3100 50  0001 C CNN
 F 3 "~" H 5800 3100 50  0001 C CNN
 	1    5800 3100
@@
 F 0 "R17" H 6670 3146 50  0000 L CNN
 F 1 "0" H 6670 3055 50  0000 L CNN
-F 2 "Resistors_SMD:R_2010_HandSoldering" V 6530 3100 50  0001 C CNN
+F 2 "mod:R_2010_HandSoldering" V 6530 3100 50  0001 C CNN
 F 3 "~" H 6600 3100 50  0001 C CNN
 	1    6600 3100
@@
 F 0 "R20" H 5670 2596 50  0000 L CNN
 F 1 "820" H 5670 2505 50  0000 L CNN
-F 2 "Resistors_SMD:R_1206_HandSoldering" V 5530 2550 50  0001 C CNN
+F 2 "mod:R_1206_HandSoldering" V 5530 2550 50  0001 C CNN
 F 3 "~" H 5600 2550 50  0001 C CNN
 	1    5600 2550
